File: PCB-RevB/RobotLegoController/01-Microcontroller and Extras.kicad_sch (KiCad schematic)
At the start: 102 parts, among them J1 DF11-10DP-2DSA, J2 Raspberry_Pi_2_3, Q1 BSS84, Q2 BSS84, SW1 SW_Omron_B3FS, SW2 SW_Omron_B3FS, SW5 SW_Omron_B3FS, U1 LSM6DSL, U2 STM32L496ZGTx, U3 SSD1306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

Commit message: Finish updating schematic REV B
Parts:
- R21: renamed from R?; now fitted
- R26: renamed from R?; now not fitted
- gave numbers to parts that had none: 10
- renumbered C50 to C9
Connections:
- net 5VON: now reaches U2.59 (PE8)
- net 9VON: now reaches U2.60 (PE9)
- no-connect marks 35 -> 33
Other:
- note added: "Configured OD"
