File: PCB-RevB/RobotLegoController/02-System Power Supply and USB.kicad_sch (KiCad schematic)
At the start: 164 parts, among them J3 USB_C_Receptacle_USB2.0, J4 Conn_01x02, Q13 2N7002, Q3 BSS84, Q37 2N7002, Q4 2N7002, SW5 SW_Omron_B3FS, U5 FUSB302B01MPX, U6 BQ25601, U7 AP2127K-3.3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

Commit message: Finish updating schematic REV B
Parts:
- removed F1, F2: 8V 2A, Resistor_SMD:R_1812_4532Metric, symbol Device:Polyfuse
- added C183, C184: 330p, Capacitor_SMD:C_0402_1005Metric, symbol Device:C_Small
- added Q14, Q21: Si2371EDS, Package_TO_SOT_SMD:SOT-23, symbol Transistor_FET:Si2371EDS
- added R156, R158: 29K4, Resistor_SMD:R_0402_1005Metric, symbol Device:R_US
- added R157, R159: 2K4, Resistor_SMD:R_0402_1005Metric, symbol Device:R_US
- added R246, R247: 330, Resistor_SMD:R_0402_1005Metric, symbol Device:R_US
- R63: value 51K -> 10K; Digi https://www.digikey.co.uk/en/products/detail/stackpole-elec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 -> (none)
- R64: value 51K -> 29K4
- gave numbers to parts that had none: 15
- renumbered SW5 to SW3
Connections:
- net +4V: now also R64.2, Q14.2 (S), Q21.2 (S), R158.2
- net 5BOOSTIN: now also Q14.3 (D)
- net 9BOOSTIN: now also Q21.3 (D)
- net GND: now also R246.2, R247.2
- net at D12.2 (A), L3.2, U9.8 (SW): now also C183.1
- net at R64.1: now also Q14.1 (G), R157.2; no longer C85.1
- net at D11.2 (A), L2.2, U8.8 (SW): now also C184.1
- net at C83.1, U9.4 (COMP): now also R156.2; no longer R64.2
- new net: C85.1, R156.1
- new net: Q21.1 (G), R158.1, R159.2
- new net: C184.2, R247.1
- new net: C183.2, R246.1
- new net 5VON: R157.1
- new net 9VON: R159.1
Other:
- moved on the sheet: TP40, TP41
