File: PCB-RevB/RobotLegoController/03-System Inputs A.kicad_sch (KiCad schematic)
At the start: 119 parts

Commit message: Finish updating schematic REV B
Parts:
- J7, J8: renamed from J?; footprint Connector_RJ:RJ12_Amphenol_54601 -> Connector_RJ:RJ25_Wayconn_MJEA-660X1_Horizontal
- gave numbers to parts that had none: 111
