File: PCB-RevB/RobotLegoController/05-System Outputs A.kicad_sch (KiCad schematic)
At the start: 109 parts, among them U12 LMV324, U13 SN74LVC1G14DBV, U14 SN74LVC1G14DBV, U15 SN74LVC1G14DBV, U16 SN74LVC1G14DBV, U17 DRV8833PWP

Commit message: Finish updating schematic REV B
Parts:
- removed D? (x4): BAT54S, Package_TO_SOT_SMD:SOT-23, symbol Diode:BAT54S
- added R241, R244, R248, R249: 4K7, Resistor_SMD:R_0402_1005Metric, symbol Device:R_US
- J11, J12: renamed from J?; footprint Connector_RJ:RJ12_Amphenol_54601 -> Connector_RJ:RJ25_Wayconn_MJEA-660X1_Horizontal
- gave numbers to parts that had none: 50
Connections:
- net MOTORA_PIN5: now also R241.1
- net MOTORA_PIN5_ENC: no longer Q29.3 (D)
- net MOTORA_PIN6: now also R244.1
- net MOTORA_PIN6_ENC: no longer Q31.3 (D)
- net MOTORB_PIN5: now also R249.1
- net MOTORB_PIN5_ENC: no longer Q30.3 (D)
- net MOTORB_PIN6: now also R248.1
- net MOTORB_PIN6_ENC: no longer Q32.3 (D)
- new net: Q31.3 (D), R244.2
- new net: Q29.3 (D), R241.2
- new net: Q32.3 (D), R248.2
- new net: Q30.3 (D), R249.2
Other:
- note added: "FC=10KHz"
- moved on the sheet: C133, C134, C138, C139, Q29, Q30, Q31, Q32, R174, R176, R177, R178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
