File: PCB-RevB/RobotLegoController/RobotLegoController.kicad_sch (KiCad schematic)
At the start: 11 parts

Commit message: Finish updating schematic REV B
Other:
- note added: "1 0"
- note added: "PCB Rev B"
