File: PCB-RevB/RobotLegoController/RobotLegoController.kicad_pcb (KiCad board)
At the start: 4 copper layers, 80 x 105 mm, 725 parts, among them J1 DF11-10DP-2DSA, J10 RJ12, J11 RJ12, J12 RJ12, J13 RJ12, J14 RJ12, J2 Raspberry_Pi_2_3, J3 USB_C_Receptacle_USB2.0, J4 Conn_01x02, J7 RJ12, J8 RJ12, J9 RJ12, Q1 BSS84, Q10 BSS84, Q11 BSS84, Q12 BSS84, Q13 2N7002, Q15 2N7002, Q16 2N7002, Q17 BSS84, Q18 BSS84, Q19 2N7002, Q2 BSS84, Q20 2N7002, Q27 2N7002, Q28 2N7002, Q29 2N7002, Q3 BSS84, Q30 2N7002, Q31 2N7002, Q32 2N7002, Q33 2N7002, Q34 2N7002, Q35 2N7002, Q36 2N7002, Q37 2N7002, Q4 2N7002, Q5 BSS84, Q6 BSS84, Q7 2N7002, Q8 2N7002, Q9 BSS84, SW1 SW_Omron_B3FS, SW2 SW_Omron_B3FS, SW3 SW_Omron_B3FS, SW5 SW_Omron_B3FS, U1 LSM6DSL, U10 LMV324, U11 LMV324, U12 LMV324, U13 SN74LVC1G14DBV, U14 SN74LVC1G14DBV, U15 SN74LVC1G14DBV, U16 SN74LVC1G14DBV, U17 DRV8833PWP, U18 LMV324, U19 SN74LVC1G14DBV, U2 STM32L496ZGTx, U20 SN74LVC1G14DBV, U21 SN74LVC1G14DBV, U22 SN74LVC1G14DBV, U23 DRV8833PWP, U3 SSD1306, U4 W25X40CLSS, U5 FUSB302B01MPX, U6 BQ25601, U7 AP2127K-3.3, U8 PAM2423AECADJR, U9 PAM2423AECADJR, Y2 8Z-24.000MAAJ-T

Commit message: More pcb routing for rev b
Parts:
- removed D43, D44, D47, D48, D55, D56, D59, D60: BAT54S, Package_TO_SOT_SMD:SOT-23
- removed F1, F2: 8V 2A, Resistor_SMD:R_1812_4532Metric
- added C183: 330p, Capacitor_SMD:C_0402_1005Metric, F.Cu at (145.3, 59.0)
- added C184: 330p, Capacitor_SMD:C_0402_1005Metric, F.Cu at (146.4, 73.1)
- added Q14: Si2371EDS, Package_TO_SOT_SMD:SOT-23, F.Cu at (135.5, 76.4)
- added Q21: Si2371EDS, Package_TO_SOT_SMD:SOT-23, F.Cu at (135.5, 61.9)
- added R155: 4K7, Resistor_SMD:R_0402_1005Metric, F.Cu at (171.0, 41.5)
- added R156: 29K4, Resistor_SMD:R_0402_1005Metric, F.Cu at (138.8, 69.6)
- added R157: 2K4, Resistor_SMD:R_0402_1005Metric, F.Cu at (136.0, 74.2)
- added R158: 29K4, Resistor_SMD:R_0402_1005Metric, F.Cu at (134.1, 59.4)
- added R159: 2K4, Resistor_SMD:R_0402_1005Metric, F.Cu at (136.0, 59.4)
- added R241: 4K7, Resistor_SMD:R_0402_1005Metric, F.Cu at (144.6, 54.4)
- added R244: 4K7, Resistor_SMD:R_0402_1005Metric, F.Cu at (136.9, 53.9)
- added R245: 4K7, Resistor_SMD:R_0402_1005Metric, F.Cu at (175.1, 39.6)
- added R246: 330, Resistor_SMD:R_0402_1005Metric, F.Cu at (143.4, 59.0)
- added R247: 330, Resistor_SMD:R_0402_1005Metric, F.Cu at (144.5, 73.1)
- added R248: 4K7, Resistor_SMD:R_0402_1005Metric, F.Cu at (156.0, 44.1)
- added R249: 4K7, Resistor_SMD:R_0402_1005Metric, F.Cu at (154.2, 45.1)
- added R250: 4K7, Resistor_SMD:R_0402_1005Metric, F.Cu at (185.6, 40.1)
- added R251: 4K7, Resistor_SMD:R_0402_1005Metric, F.Cu at (189.2, 41.4)
- R63: value 51K -> 10K
- R64: value 51K -> 29K4
- TP43: moved to B.Cu
- moved Q31 31.6 mm to (139.0, 55.9)
- moved Q29 27.4 mm to (142.4, 55.9), turned to 90 degrees
- moved Q30 25.2 mm to (157.3, 55.7), turned to 90 degrees
- moved Q32 23.6 mm to (160.4, 55.3), turned to -90 degrees
- moved Q33 21.1 mm to (173.4, 55.3), turned to 90 degrees
- moved Q34 20.2 mm to (186.8, 55.5), turned to 90 degrees
- moved Q35 19.9 mm to (176.3, 55.3), turned to -90 degrees
- moved Q36 19.0 mm to (189.9, 55.3), turned to -90 degrees
- moved J7 17.1 mm to (148.8, 128.1)
- moved J8 17.1 mm to (164.7, 128.1)
- moved J10 17.1 mm to (196.4, 128.1)
- moved J9 17.1 mm to (180.4, 128.1)
- moved TP87 9.39 mm to (175.3, 134.1)
- moved TP65 9.30 mm to (159.5, 134.1)
- moved TP89 9.26 mm to (191.4, 134.1)
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Connections:
- Q29 pad 3: /05-System Outputs A/MOTORA_PIN5_ENC -> Net-(Q29-D)
- Q30 pad 3: /05-System Outputs A/MOTORB_PIN5_ENC -> Net-(Q30-D)
- Q31 pad 3: /05-System Outputs A/MOTORA_PIN6_ENC -> Net-(Q31-D)
- Q32 pad 3: /05-System Outputs A/MOTORB_PIN6_ENC -> Net-(Q32-D)
- Q33 pad 3: /06-System Outputs B/MOTORC_PIN5_ENC -> Net-(Q33-D)
- Q34 pad 3: /06-System Outputs B/MOTORD_PIN5_ENC -> Net-(Q34-D)
- Q35 pad 3: /06-System Outputs B/MOTORC_PIN6_ENC -> Net-(Q35-D)
- Q36 pad 3: /06-System Outputs B/MOTORD_PIN6_ENC -> Net-(Q36-D)
- R64 pad 1: Net-(C85-Pad1) -> Net-(Q14-G)
- R64 pad 2: Net-(U9-COMP) -> +4V
- U2 pad 59: unconnected-(U2-PE8-Pad59) -> 5VON
- U2 pad 60: unconnected-(U2-PE9-Pad60) -> 9VON
Routing:
- net 9VON: track 0.00 -> 77.0 mm, vias 0 -> 3
- net 5VON: track 0.00 -> 74.5 mm, vias 0 -> 3
- net +5V: track 608.5 -> 554.5 mm, vias 54 -> 56
- net /03-System Inputs A/INPUT1_PIN1: track 20.1 -> 29.6 mm, vias 0 -> 1
- net +4V: track 66.6 -> 74.9 mm
- net /03-System Inputs A/INPUT2_PIN1: track 26.1 -> 34.3 mm, vias 0 -> 1
- net GND: track 595.2 -> 587.2 mm, vias 324 -> 317
- net +3.3V: track 709.8 -> 717.7 mm
- net /05-System Outputs A/MOTORA_PIN6_ENC: track 46.2 -> 38.6 mm
- net /05-System Outputs A/MOTORB_PIN6_ENC: track 45.5 -> 39.2 mm
- net /06-System Outputs B/MOTORD_PIN6_ENC: track 30.7 -> 24.6 mm
- net Net-(C94-Pad2): track 8.92 -> 15.0 mm, vias 0 -> 2
- net /03-System Inputs A/INPUT1_PIN6: track 23.1 -> 28.9 mm, vias 0 -> 1
- net +9V: track 242.0 -> 236.6 mm
- net /04-System Inputs B/INPUT3_PIN1: track 28.9 -> 34.1 mm, vias 0 -> 1
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