File: PCB-RevB/RobotLegoController/RobotLegoController.kicad_pcb (KiCad board)
At the start: 4 copper layers, 80 x 105 mm, 732 parts, among them J1 DF11-10DP-2DSA, J10 RJ12, J11 RJ12, J12 RJ12, J13 RJ12, J14 RJ12, J2 Raspberry_Pi_2_3, J3 USB_C_Receptacle_USB2.0, J4 Conn_01x02, J7 RJ12, J8 RJ12, J9 RJ12, Q1 BSS84, Q10 BSS84, Q11 BSS84, Q12 BSS84, Q13 2N7002, Q14 Si2371EDS, Q15 2N7002, Q16 2N7002, Q17 BSS84, Q18 BSS84, Q19 2N7002, Q2 BSS84, Q20 2N7002, Q21 Si2371EDS, Q27 2N7002, Q28 2N7002, Q29 2N7002, Q3 BSS84, Q30 2N7002, Q31 2N7002, Q32 2N7002, Q33 2N7002, Q34 2N7002, Q35 2N7002, Q36 2N7002, Q37 2N7002, Q4 2N7002, Q5 BSS84, Q6 BSS84, Q7 2N7002, Q8 2N7002, Q9 BSS84, SW1 SW_Omron_B3FS, SW2 SW_Omron_B3FS, SW3 SW_Omron_B3FS, SW5 SW_Omron_B3FS, U1 LSM6DSL, U10 LMV324, U11 LMV324, U12 LMV324, U13 SN74LVC1G14DBV, U14 SN74LVC1G14DBV, U15 SN74LVC1G14DBV, U16 SN74LVC1G14DBV, U17 DRV8833PWP, U18 LMV324, U19 SN74LVC1G14DBV, U2 STM32L496ZGTx, U20 SN74LVC1G14DBV, U21 SN74LVC1G14DBV, U22 SN74LVC1G14DBV, U23 DRV8833PWP, U3 SSD1306, U4 W25X40CLSS, U5 FUSB302B01MPX, U6 BQ25601, U7 AP2127K-3.3, U8 PAM2423AECADJR, U9 PAM2423AECADJR, Y2 8Z-24.000MAAJ-T

Commit message: More work on pcb layout
Parts:
- moved C168 29.6 mm to (194.6, 27.6)
- moved R240 29.6 mm to (194.6, 26.7)
- moved C170 28.6 mm to (199.3, 26.1)
- moved D54 28.6 mm to (194.1, 20.9)
- moved D58 28.6 mm to (192.2, 20.9)
- moved C156 28.6 mm to (194.1, 21.9)
- moved C162 28.6 mm to (192.2, 21.9)
- moved R210 28.6 mm to (194.1, 23.8)
- moved R212 28.6 mm to (194.1, 24.8)
- moved R226 28.6 mm to (192.2, 24.8)
- moved R238 28.6 mm to (199.3, 24.2)
- moved U22 28.6 mm to (201.9, 27.5)
- moved R216 28.6 mm to (194.1, 22.8)
- moved R224 28.6 mm to (192.2, 23.8)
- moved R230 28.6 mm to (192.2, 22.9)
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Routing:
- net +3.3V: track 717.7 -> 612.2 mm, vias 86 -> 80
- net /05-System Outputs A/MOTORA_PIN2: track 24.1 -> 67.0 mm, vias 2 -> 3
- net /05-System Outputs A/MOTORB_PIN6_ENC: track 39.2 -> 0.71 mm, vias 2 -> 0
- net +5V: track 554.5 -> 525.5 mm, vias 56 -> 51
- net Net-(Q31-G): track 2.69 -> 29.3 mm
- net /05-System Outputs A/MOTORB_PIN5_ENC: track 32.8 -> 11.0 mm, vias 2 -> 0
- net GND: track 577.9 -> 556.5 mm, vias 317 -> 297
- net /06-System Outputs B/MOTORD_PIN5_ENC: track 38.3 -> 22.8 mm, vias 2 -> 0
- net /06-System Outputs B/MOTORC_PIN5_ENC: track 36.7 -> 21.3 mm, vias 2 -> 0
- net Net-(C157-Pad2): track 4.09 -> 19.4 mm, vias 0 -> 1
- net Net-(C135-Pad2): track 4.09 -> 19.4 mm, vias 0 -> 1
- net Net-(C132-Pad2): track 4.09 -> 19.4 mm, vias 0 -> 1
- net Net-(C160-Pad2): track 4.09 -> 19.4 mm, vias 0 -> 1
- net MOTORB_PIN5_ENCODER: track 74.9 -> 60.6 mm
- net /05-System Outputs A/MOTORB_PIN2: track 17.9 -> 4.71 mm, vias 2 -> 1
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